Commit message: URDF model and gazebo simulation for raspicam

File: turtlebot3_description/urdf/turtlebot3_burger.gazebo.xacro (robot description, xacro)
@@ -120,3 +120,40 @@
     </sensor>
   </gazebo>
+  <gazebo reference="raspicam_link">
+    <sensor type="camera" name="raspicam">
+      <update_rate>30.0</update_rate>
+      <camera name="raspicam">
+        <horizontal_fov>1.085595</horizontal_fov>
+        <vertical_fov>0.8517207</vertical_fov>
+        <image>
+          <width>1280</width>
+          <height>960</height>
+          <format>R8G8B8</format>
+        </image>
+        <clip>
+          <near>0.02</near>
+          <far>300</far>
+        </clip>
+        <noise>
+          <type>gaussian</type>
+          <mean>0.0</mean>
+          <stddev>0.007</stddev>
+        </noise>
+      </camera>
+      <plugin name="camera_controller" filename="libgazebo_ros_camera.so">
+        <alwaysOn>true</alwaysOn>
+        <updateRate>0.0</updateRate>
+        <cameraName>raspicam_node</cameraName>
+        <imageTopicName>image/compressed</imageTopicName>
+        <cameraInfoTopicName>camera_info</cameraInfoTopicName>
+        <frameName>raspicam_link</frameName>
+        <hackBaseline>0.07</hackBaseline>
+        <distortionK1>0.0</distortionK1>
+        <distortionK2>0.0</distortionK2>
+        <distortionK3>0.0</distortionK3>
+        <distortionT1>0.0</distortionT1>
+        <distortionT2>0.0</distortionT2>
+      </plugin>
+    </sensor>
+  </gazebo>
 </robot>

File: turtlebot3_description/urdf/turtlebot3_burger.urdf.xacro (robot description, xacro)
@@ -140,3 +140,17 @@
     </inertial>
   </link>
+  <joint name="raspicam_joint" type="fixed">
+    <parent link="base_link" />
+    <child link="raspicam_link" />
+    <origin xyz="0.04 0 0.115" rpy="0 0 0" />
+  </joint>
+  <link name="raspicam_link">
+    <visual>
+      <origin xyz="0 0 0.005" rpy="0 0 0" />
+      <geometry>
+        <box size="0.003 0.03 0.025" />
+      </geometry>
+      <material name="dark" />
+    </visual>
+  </link>
 </robot>
